Commit message: merged master into shah_control_rl

File: soccer_description/models/parameters.xacro (robot description, xacro)
@@ -13,4 +13,10 @@
     <xacro:property name="AX12_TORQUE" value="1.5"/>
     <xacro:property name="AX12_VELOCITY" value="1"/>
+    <material name="white">
+        <color rgba="1.0 1.0 1.0 1.0"/>
+    </material>
+    <material name="black">
+        <color rgba="0.0 0.0 0.0 1.0"/>
+    </material>
     <material name="silver">
         <color rgba="0.7 0.7 0.7 1.0"/>
@@ -34,6 +40,3 @@
         <color rgba="0.0 0.7 0.7 1.0"/>
     </material>
-    <material name="black">
-        <color rgba="0.2 0.2 0.2 1.0"/>
-    </material>
 </robot>

File: soccer_description/models/soccerbot_stl.urdf (robot description, URDF)
Before this commit: robot soccerbot, 21 links, 20 joints
Joints:
- joint /torso_imu: origin xyz=0.1 0 0.0075 rpy=0 0 0 -> xyz=0.0 0 0.000 rpy=0 0 0
